File: hardware/driver-board/motor_control.kicad_sch (KiCad schematic)
At the start: 16 parts, among them J3 CONN_MOTOR_R, J4 CONN_MOTOR_L, U3 DRV8838, U4 DRV8838

Commit message: Finalize Rev A PCB and hardware docs
Parts:
- R12, R13: JLCPCB (none) -> C25741
Changed lines of the file:
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@@
 			)
 		)
-		(property "JLCPCB" ""
+		(property "JLCPCB" "C25741"
 			(at 152.4 138.43 0)
 			(hide yes)
@@
 			)
 		)
-		(property "JLCPCB" ""
+		(property "JLCPCB" "C25741"
 			(at 100.33 73.66 0)
 			(hide yes)
