File: hardware/driver-board/power.kicad_sch (KiCad schematic)
At the start: 26 parts, among them Q1 AO3401A, Q2 AO4407A, SW2 SK-3296S-01-L2, U5 LMR51430XDDCR

Commit message: Refine driver board placement and motor power checks
Parts:
- R16: footprint Resistor_SMD:R_0603_1608Metric -> Resistor_SMD:R_0402_1005Metric; JLCPCB C25803 -> (none)
- R17: footprint Resistor_SMD:R_0603_1608Metric -> Resistor_SMD:R_0402_1005Metric; JLCPCB C4216 -> (none)
Changed lines of the file:
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@@
 			)
 		)
-		(property "Footprint" "Resistor_SMD:R_0603_1608Metric"
+		(property "Footprint" "Resistor_SMD:R_0402_1005Metric"
 			(at 256.54 63.5 0)
 			(hide yes)
@@
 			)
 		)
-		(property "JLCPCB" "C4216"
+		(property "JLCPCB" ""
 			(at 256.54 63.5 0)
 			(hide yes)
@@
 			)
 		)
-		(property "Footprint" "Resistor_SMD:R_0603_1608Metric"
+		(property "Footprint" "Resistor_SMD:R_0402_1005Metric"
 			(at 256.54 48.26 0)
 			(hide yes)
@@
 			)
 		)
-		(property "JLCPCB" "C25803"
+		(property "JLCPCB" ""
 			(at 256.54 48.26 0)
 			(hide yes)

Commit message: Refine Rev A PCB placement and decoupling
Parts:
- R18: footprint Resistor_SMD:R_0603_1608Metric -> Resistor_SMD:R_0402_1005Metric; JLCPCB C25803 -> (none)
- R19: footprint Resistor_SMD:R_0603_1608Metric -> Resistor_SMD:R_0402_1005Metric; JLCPCB C137768 -> (none)
Connections:
- net REG_SW: now reaches C19.2, L1.1, U5.2 (SW)
Changed lines of the file:
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@@
+		)
+	)
+	(label "REG_SW"
+		(at 140.97 115.57 0)
+		(effects
+			(font
+				(size 1.27 1.27)
+			)
+			(justify left bottom)
 		)
 	)
@@
 			)
 		)
-		(property "Footprint" "Resistor_SMD:R_0603_1608Metric"
+		(property "Footprint" "Resistor_SMD:R_0402_1005Metric"
 			(at 155.702 123.19 90)
 			(hide yes)
@@
 			)
 		)
-		(property "Description" "-55℃~+155℃ 100kΩ 100mW 75V Thick Film Resistor ±1%"
+		(property "Description" "LMR51430 upper feedback resistor (+3V3 to FB): 100kΩ, ±1% or better, low temperature coefficient; place close to U5 FB and route away from the SW node and inductor; standard 0402 power rating is sufficient"
 			(at 157.48 123.19 0)
 			(hide yes)
@@
 			)
 		)
-		(property "JLCPCB" "C25803"
+		(property "JLCPCB" ""
 			(at 157.48 123.19 0)
 			(hide yes)
@@
 			)
 		)
-		(property "Footprint" "Resistor_SMD:R_0603_1608Metric"
+		(property "Footprint" "Resistor_SMD:R_0402_1005Metric"
 			(at 155.702 135.89 90)
 			(hide yes)
@@
 			)
 		)
-		(property "Description" "100mW 22.1kΩ 75V Thick Film Resistor ±1%"
+		(property "Description" "LMR51430 lower feedback resistor (FB to GND): 22.1kΩ, ±1% or better, low temperature coefficient; place close to U5 FB with a quiet ground return and route away from the SW node and inductor; standard 0402 power rating is sufficient"
 			(at 157.48 135.89 0)
 			(hide yes)
@@
 			)
 		)
-		(property "JLCPCB" "C137768"
+		(property "JLCPCB" ""
 			(at 157.48 135.89 0)
 			(hide yes)

Commit message: Refine driver board layout and 3D models
Changed lines of the file:
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@@
 	)
 	(label "REG_SW"
-		(at 140.97 115.57 0)
+		(at 139.7 115.57 0)
 		(effects
 			(font

Commit message: Finalize Rev A PCB and hardware docs
Parts:
- R16, R18: JLCPCB (none) -> C25741
- R17: JLCPCB (none) -> C25779
- R19: JLCPCB (none) -> C43473
Changed lines of the file:
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@@
 			)
 		)
-		(property "JLCPCB" ""
+		(property "JLCPCB" "C25741"
 			(at 157.48 123.19 0)
 			(hide yes)
@@
 			)
 		)
-		(property "JLCPCB" ""
+		(property "JLCPCB" "C25779"
 			(at 256.54 63.5 0)
 			(hide yes)
@@
 			)
 		)
-		(property "JLCPCB" ""
+		(property "JLCPCB" "C43473"
 			(at 157.48 135.89 0)
 			(hide yes)
@@
 			)
 		)
-		(property "JLCPCB" ""
+		(property "JLCPCB" "C25741"
 			(at 256.54 48.26 0)
 			(hide yes)
